File: mwpc/mwpc.kicad_pcb (KiCad board)
At the start: 2 copper layers, 132 parts, among them X1 MWPC_HVT, X2 MWPC_HVT, X3 MWPC_HVT, X4 MWPC_HVT

Commit message: Rearrange the components on the PCB.
Parts:
- removed X2, X4: MWPC_HVT, mwpc:MWPC_HVT_SMD
- added REF**: Terminal, mwpc:Terminal, F.Cu at (60.0, 31.4)
- added REF**: Terminal, mwpc:Terminal, F.Cu at (65.0, 162.5)
- added locked: MWPC_HVT, mwpc:MWPC_HVT_SMD, F.Cu at (100.0, 82.0)
- added locked: MWPC_HVT, mwpc:MWPC_HVT_SMD, F.Cu at (100.0, 146.0)
- moved R105 240.8 mm to (85.0, 139.5)
- moved R121 239.0 mm to (85.0, 155.5)
- moved R126 238.1 mm to (93.0, 160.5)
- moved R127 236.4 mm to (85.0, 161.5)
- moved R97 235.0 mm to (85.0, 131.5)
- moved R119 234.7 mm to (85.0, 153.5)
- moved R61 227.8 mm to (85.0, 95.5)
- moved R114 227.4 mm to (93.0, 148.5)
- moved R117 227.2 mm to (85.0, 151.5)
- moved R79 226.7 mm to (85.0, 113.5)
- moved R90 226.4 mm to (93.0, 124.5)
- moved R109 225.8 mm to (85.0, 143.5)
- moved R120 225.7 mm to (93.0, 154.5)
- moved R106 225.5 mm to (93.0, 140.5)
- moved R124 224.8 mm to (93.0, 158.5)
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Connections:
- R100 pad 2: Net-(R100-Pad2) -> Net-(R4-Pad2)
- R101 pad 2: Net-(R101-Pad2) -> Net-(R5-Pad2)
- R102 pad 2: Net-(R102-Pad2) -> Net-(R6-Pad2)
- R103 pad 2: Net-(R103-Pad2) -> Net-(R7-Pad2)
- R104 pad 2: Net-(R104-Pad2) -> Net-(R8-Pad2)
- R105 pad 2: Net-(R105-Pad2) -> Net-(R9-Pad2)
- R106 pad 2: Net-(R106-Pad2) -> Net-(R10-Pad2)
- R107 pad 2: Net-(R107-Pad2) -> Net-(R11-Pad2)
- R108 pad 2: Net-(R108-Pad2) -> Net-(R12-Pad2)
- R109 pad 2: Net-(R109-Pad2) -> Net-(R13-Pad2)
- R110 pad 2: Net-(R110-Pad2) -> Net-(R14-Pad2)
- R111 pad 2: Net-(R111-Pad2) -> Net-(R15-Pad2)
- R112 pad 2: Net-(R112-Pad2) -> Net-(R16-Pad2)
- R113 pad 2: Net-(R113-Pad2) -> Net-(R17-Pad2)
- R114 pad 2: Net-(R114-Pad2) -> Net-(R18-Pad2)
- R115 pad 2: Net-(R115-Pad2) -> Net-(R19-Pad2)
- R116 pad 2: Net-(R116-Pad2) -> Net-(R20-Pad2)
- R117 pad 2: Net-(R117-Pad2) -> Net-(R21-Pad2)
- R118 pad 2: Net-(R118-Pad2) -> Net-(R22-Pad2)
- R119 pad 2: Net-(R119-Pad2) -> Net-(R23-Pad2)
- R120 pad 2: Net-(R120-Pad2) -> Net-(R24-Pad2)
- R121 pad 2: Net-(R121-Pad2) -> Net-(R25-Pad2)
- R122 pad 2: Net-(R122-Pad2) -> Net-(R26-Pad2)
- R123 pad 2: Net-(R123-Pad2) -> Net-(R27-Pad2)
- R124 pad 2: Net-(R124-Pad2) -> Net-(R28-Pad2)
- R125 pad 2: Net-(R125-Pad2) -> Net-(R29-Pad2)
- R126 pad 2: Net-(R126-Pad2) -> Net-(R30-Pad2)
- R127 pad 2: Net-(R127-Pad2) -> Net-(R31-Pad2)
- R128 pad 2: Net-(R128-Pad2) -> Net-(R32-Pad2)
- R33 pad 2: Net-(R33-Pad2) -> Net-(R1-Pad2)
- R34 pad 2: Net-(R34-Pad2) -> Net-(R2-Pad2)
- R35 pad 2: Net-(R35-Pad2) -> Net-(R3-Pad2)
- R36 pad 2: Net-(R36-Pad2) -> Net-(R4-Pad2)
- R37 pad 2: Net-(R37-Pad2) -> Net-(R5-Pad2)
- R38 pad 2: Net-(R38-Pad2) -> Net-(R6-Pad2)
- R39 pad 2: Net-(R39-Pad2) -> Net-(R7-Pad2)
- R40 pad 2: Net-(R40-Pad2) -> Net-(R8-Pad2)
- R41 pad 2: Net-(R41-Pad2) -> Net-(R9-Pad2)
- R42 pad 2: Net-(R42-Pad2) -> Net-(R10-Pad2)
- R43 pad 2: Net-(R43-Pad2) -> Net-(R11-Pad2)
- R44 pad 2: Net-(R44-Pad2) -> Net-(R12-Pad2)
- R45 pad 2: Net-(R45-Pad2) -> Net-(R13-Pad2)
- R46 pad 2: Net-(R46-Pad2) -> Net-(R14-Pad2)
- R47 pad 2: Net-(R47-Pad2) -> Net-(R15-Pad2)
- R48 pad 2: Net-(R48-Pad2) -> Net-(R16-Pad2)
- R49 pad 2: Net-(R49-Pad2) -> Net-(R17-Pad2)
- R50 pad 2: Net-(R50-Pad2) -> Net-(R18-Pad2)
- R51 pad 2: Net-(R51-Pad2) -> Net-(R19-Pad2)
- R52 pad 2: Net-(R52-Pad2) -> Net-(R20-Pad2)
- R53 pad 2: Net-(R53-Pad2) -> Net-(R21-Pad2)
- R54 pad 2: Net-(R54-Pad2) -> Net-(R22-Pad2)
- R55 pad 2: Net-(R55-Pad2) -> Net-(R23-Pad2)
- R56 pad 2: Net-(R56-Pad2) -> Net-(R24-Pad2)
- R57 pad 2: Net-(R57-Pad2) -> Net-(R25-Pad2)
- R58 pad 2: Net-(R58-Pad2) -> Net-(R26-Pad2)
- R59 pad 2: Net-(R59-Pad2) -> Net-(R27-Pad2)
- R60 pad 2: Net-(R60-Pad2) -> Net-(R28-Pad2)
- R61 pad 2: Net-(R61-Pad2) -> Net-(R29-Pad2)
- R62 pad 2: Net-(R62-Pad2) -> Net-(R30-Pad2)
- R63 pad 2: Net-(R63-Pad2) -> Net-(R31-Pad2)
- R64 pad 2: Net-(R64-Pad2) -> Net-(R32-Pad2)
- R65 pad 2: Net-(R65-Pad2) -> Net-(R1-Pad2)
- R66 pad 2: Net-(R66-Pad2) -> Net-(R2-Pad2)
- R67 pad 2: Net-(R67-Pad2) -> Net-(R3-Pad2)
- R68 pad 2: Net-(R68-Pad2) -> Net-(R4-Pad2)
- R69 pad 2: Net-(R69-Pad2) -> Net-(R5-Pad2)
- R70 pad 2: Net-(R70-Pad2) -> Net-(R6-Pad2)
- R71 pad 2: Net-(R71-Pad2) -> Net-(R7-Pad2)
- R72 pad 2: Net-(R72-Pad2) -> Net-(R8-Pad2)
- R73 pad 2: Net-(R73-Pad2) -> Net-(R9-Pad2)
- R74 pad 2: Net-(R74-Pad2) -> Net-(R10-Pad2)
- R75 pad 2: Net-(R75-Pad2) -> Net-(R11-Pad2)
- R76 pad 2: Net-(R76-Pad2) -> Net-(R12-Pad2)
- R77 pad 2: Net-(R77-Pad2) -> Net-(R13-Pad2)
- R78 pad 2: Net-(R78-Pad2) -> Net-(R14-Pad2)
- R79 pad 2: Net-(R79-Pad2) -> Net-(R15-Pad2)
- R80 pad 2: Net-(R80-Pad2) -> Net-(R16-Pad2)
- R81 pad 2: Net-(R81-Pad2) -> Net-(R17-Pad2)
- R82 pad 2: Net-(R82-Pad2) -> Net-(R18-Pad2)
- R83 pad 2: Net-(R83-Pad2) -> Net-(R19-Pad2)
- R84 pad 2: Net-(R84-Pad2) -> Net-(R20-Pad2)
- R85 pad 2: Net-(R85-Pad2) -> Net-(R21-Pad2)
- R86 pad 2: Net-(R86-Pad2) -> Net-(R22-Pad2)
- R87 pad 2: Net-(R87-Pad2) -> Net-(R23-Pad2)
- R88 pad 2: Net-(R88-Pad2) -> Net-(R24-Pad2)
- R89 pad 2: Net-(R89-Pad2) -> Net-(R25-Pad2)
- R90 pad 2: Net-(R90-Pad2) -> Net-(R26-Pad2)
- R91 pad 2: Net-(R91-Pad2) -> Net-(R27-Pad2)
- R92 pad 2: Net-(R92-Pad2) -> Net-(R28-Pad2)
- R93 pad 2: Net-(R93-Pad2) -> Net-(R29-Pad2)
- R94 pad 2: Net-(R94-Pad2) -> Net-(R30-Pad2)
- R95 pad 2: Net-(R95-Pad2) -> Net-(R31-Pad2)
- R96 pad 2: Net-(R96-Pad2) -> Net-(R32-Pad2)
- R97 pad 2: Net-(R97-Pad2) -> Net-(R1-Pad2)
- R98 pad 2: Net-(R98-Pad2) -> Net-(R2-Pad2)
- R99 pad 2: Net-(R99-Pad2) -> Net-(R3-Pad2)
- X3 pad 1: Net-(R65-Pad2) -> Net-(R1-Pad2)
- X3 pad 10: Net-(R74-Pad2) -> Net-(R10-Pad2)
- X3 pad 11: Net-(R75-Pad2) -> Net-(R11-Pad2)
- X3 pad 12: Net-(R76-Pad2) -> Net-(R12-Pad2)
- X3 pad 13: Net-(R77-Pad2) -> Net-(R13-Pad2)
- X3 pad 14: Net-(R78-Pad2) -> Net-(R14-Pad2)
- X3 pad 15: Net-(R79-Pad2) -> Net-(R15-Pad2)
- X3 pad 16: Net-(R80-Pad2) -> Net-(R16-Pad2)
- X3 pad 17: Net-(R81-Pad2) -> Net-(R17-Pad2)
- X3 pad 18: Net-(R82-Pad2) -> Net-(R18-Pad2)
- X3 pad 19: Net-(R83-Pad2) -> Net-(R19-Pad2)
- X3 pad 2: Net-(R66-Pad2) -> Net-(R2-Pad2)
- X3 pad 20: Net-(R84-Pad2) -> Net-(R20-Pad2)
- X3 pad 21: Net-(R85-Pad2) -> Net-(R21-Pad2)
- X3 pad 22: Net-(R86-Pad2) -> Net-(R22-Pad2)
- X3 pad 23: Net-(R87-Pad2) -> Net-(R23-Pad2)
- X3 pad 24: Net-(R88-Pad2) -> Net-(R24-Pad2)
- X3 pad 25: Net-(R89-Pad2) -> Net-(R25-Pad2)
- X3 pad 26: Net-(R90-Pad2) -> Net-(R26-Pad2)
- X3 pad 27: Net-(R91-Pad2) -> Net-(R27-Pad2)
- X3 pad 28: Net-(R92-Pad2) -> Net-(R28-Pad2)
- X3 pad 29: Net-(R93-Pad2) -> Net-(R29-Pad2)
- X3 pad 3: Net-(R67-Pad2) -> Net-(R3-Pad2)
- X3 pad 30: Net-(R94-Pad2) -> Net-(R30-Pad2)
- X3 pad 31: Net-(R95-Pad2) -> Net-(R31-Pad2)
- X3 pad 32: Net-(R96-Pad2) -> Net-(R32-Pad2)
- X3 pad 4: Net-(R68-Pad2) -> Net-(R4-Pad2)
- X3 pad 5: Net-(R69-Pad2) -> Net-(R5-Pad2)
- X3 pad 6: Net-(R70-Pad2) -> Net-(R6-Pad2)
- X3 pad 7: Net-(R71-Pad2) -> Net-(R7-Pad2)
- X3 pad 8: Net-(R72-Pad2) -> Net-(R8-Pad2)
- X3 pad 9: Net-(R73-Pad2) -> Net-(R9-Pad2)
